File: hardware/kicad/nomiq/nomiq.kicad_sch (KiCad schematic)
At the start: 0 parts

Commit message: feat(sch): generate KiCad 8 hierarchical schematic from nomiq_hw.py netlist
8 sheets, 128 symbols, global-label connectivity verified against the netlist
(gen_kicad.py --check in make tools). U1/U2 pad maps per datasheet; 32 parts
flagged with placeholder pads. REQ-HW-001.

Co-Authored-By: Claude Opus 5.5 <noreply@anthropic.com>
Claude-Session: https://claude.ai/code/session_01HafD3UN2tDPG8DjCdm2PVK
Other:
- added sheet 01_power (01_power.kicad_sch)
- added sheet 02_mcu (02_mcu.kicad_sch)
- added sheet 03_radio (03_radio.kicad_sch)
- added sheet 04_audio (04_audio.kicad_sch)
- added sheet 05_camera (05_camera.kicad_sch)
- added sheet 06_display_storage (06_display_storage.kicad_sch)
- added sheet 07_ui (07_ui.kicad_sch)
- added sheet 08_stt (08_stt.kicad_sch)
- title: Nomiq — LoRa voice/text/photo messenger -> Nomiq A0 — main board
Changed lines of the file:
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@@
-(kicad_sch
-	(version 20250114)
-	(generator "eeschema")
-	(generator_version "9.0")
-	(paper "A3")
-	(title_block
-		(title "Nomiq — LoRa voice/text/photo messenger")
-		(rev "A0")
-		(comment 1 "Sheet plan: hardware/README.md")
-		(comment 2 "Pin map: docs/02-hardware-architecture.md")
-	)
-	(sheet_instances
-		(path "/"
-			(page "1")
-		)
-	)
-	(embedded_fonts no)
+(kicad_sch (version 20231120) (generator "nomiq_gen") (generator_version "8.0") (paper "A3")
+(title_block (title "Nomiq A0 — main board") (rev "A0") (comment 1 "Hierarchical sheets generated from hardware/design/nomiq_hw.py"))
+(sheet (at 30 40) (size 70 35) (fields_autoplaced yes) (stroke (width 0.1524) (type solid)) (fill (color 0 0 0 0.0000)) (property "Sheetname" "01_power" (at 30.00 39.00 0) (effects (font (size 1.27 1.27)) (justify left bottom))) (property "Sheetfile" "01_power.kicad_sch" (at 30.00 76.00 0) (effects (font (size 1.27 1.27)) (justify left top))) (instances (project "nomiq" (path "/22a78807-b768-5690-bf1c-caee3a2f8ff0" (page "2")))))
+(sheet (at 120 40) (size 70 35) (fields_autoplaced yes) (stroke (width 0.1524) (type solid)) (fill (color 0 0 0 0.0000)) (property "Sheetname" "02_mcu" (at 120.00 39.00 0) (effects (font (size 1.27 1.27)) (justify left bottom))) (property "Sheetfile" "02_mcu.kicad_sch" (at 120.00 76.00 0) (effects (font (size 1.27 1.27)) (justify left top))) (instances (project "nomiq" (path "/22a78807-b768-5690-bf1c-caee3a2f8ff0" (page "3")))))
+(sheet (at 210 40) (size 70 35) (fields_autoplaced yes) (stroke (width 0.1524) (type solid)) (fill (color 0 0 0 0.0000)) (property "Sheetname" "03_radio" (at 210.00 39.00 0) (effects (font (size 1.27 1.27)) (justify left bottom))) (property "Sheetfile" "03_radio.kicad_sch" (at 210.00 76.00 0) (effects (font (size 1.27 1.27)) (justify left top))) (instances (project "nomiq" (path "/22a78807-b768-5690-bf1c-caee3a2f8ff0" (page "4")))))
+(sheet (at 300 40) (size 70 35) (fields_autoplaced yes) (stroke (width 0.1524) (type solid)) (fill (color 0 0 0 0.0000)) (property "Sheetname" "04_audio" (at 300.00 39.00 0) (effects (font (size 1.27 1.27)) (justify left bottom))) (property "Sheetfile" "04_audio.kicad_sch" (at 300.00 76.00 0) (effects (font (size 1.27 1.27)) (justify left top))) (instances (project "nomiq" (path "/22a78807-b768-5690-bf1c-caee3a2f8ff0" (page "5")))))
+(sheet (at 30 100) (size 70 35) (fields_autoplaced yes) (stroke (width 0.1524) (type solid)) (fill (color 0 0 0 0.0000)) (property "Sheetname" "05_camera" (at 30.00 99.00 0) (effects (font (size 1.27 1.27)) (justify left bottom))) (property "Sheetfile" "05_camera.kicad_sch" (at 30.00 136.00 0) (effects (font (size 1.27 1.27)) (justify left top))) (instances (project "nomiq" (path "/22a78807-b768-5690-bf1c-caee3a2f8ff0" (page "6")))))
+(sheet (at 120 100) (size 70 35) (fields_autoplaced yes) (stroke (width 0.1524) (type solid)) (fill (color 0 0 0 0.0000)) (property "Sheetname" "06_display_storage" (at 120.00 99.00 0) (effects (font (size 1.27 1.27)) (justify left bottom))) (property "Sheetfile" "06_display_storage.kicad_sch" (at 120.00 136.00 0) (effects (font (size 1.27 1.27)) (justify left top))) (instances (project "nomiq" (path "/22a78807-b768-5690-bf1c-caee3a2f8ff0" (page "7")))))
+(sheet (at 210 100) (size 70 35) (fields_autoplaced yes) (stroke (width 0.1524) (type solid)) (fill (color 0 0 0 0.0000)) (property "Sheetname" "07_ui" (at 210.00 99.00 0) (effects (font (size 1.27 1.27)) (justify left bottom))) (property "Sheetfile" "07_ui.kicad_sch" (at 210.00 136.00 0) (effects (font (size 1.27 1.27)) (justify left top))) (instances (project "nomiq" (path "/22a78807-b768-5690-bf1c-caee3a2f8ff0" (page "8")))))
+(sheet (at 300 100) (size 70 35) (fields_autoplaced yes) (stroke (width 0.1524) (type solid)) (fill (color 0 0 0 0.0000)) (property "Sheetname" "08_stt" (at 300.00 99.00 0) (effects (font (size 1.27 1.27)) (justify left bottom))) (property "Sheetfile" "08_stt.kicad_sch" (at 300.00 136.00 0) (effects (font (size 1.27 1.27)) (justify left top))) (instances (project "nomiq" (path "/22a78807-b768-5690-bf1c-caee3a2f8ff0" (page "9")))))
+(sheet_instances (path "/" (page "1")))
 )
