File: hardware/kicad/nomiq/01_power.kicad_sch (KiCad schematic)
At the start: 40 parts, among them J1 USB-C 16P, J2 Battery JST-PH 3P (+, NTC, -), U10 TPS63802, U14 TPS22918 (STT rail), U8 BQ24074, U9 MAX17048

Commit message: feat(sch): verified pad maps and project footprint library for all 138 parts
- fplib.py: 36 footprints from the KiCad library / Espressif library (+ TFT module),
  written to lib/nomiq.pretty and checked (make tools)
- nomiq_hw.py: per-part datasheet pin->pad maps; gen_kicad checks every pad exists
  and every copper pad is mapped (0 unverified parts)
- TPS63802 -> TPS63001 (fixed 3.3 V, KiCad DRC land pattern); BQ24074 RILIM/ITERM/TMR
  corrected to datasheet constants; TCXO 1.8 V (E) variant to match DIO3 setting
- RF blocks expanded into discrete choke, 2-section low-pass, lattice balun, DC blocks
  (PE4259 ports must be DC-free) and DNP pi tuning pads
- Display: 14-pin ILI9341 module, high-side P-FET backlight switch; microSD detect pins,
  connector mounting pads, MAX98357A NC pads

REQ-PCB-001, REQ-PCB-007

Co-Authored-By: Claude Opus 5.5 <noreply@anthropic.com>
Claude-Session: https://claude.ai/code/session_01HafD3UN2tDPG8DjCdm2PVK
Parts:
- removed R10: 510k 1%, Resistor_SMD:R_0402_1005Metric, symbol nomiq:R10_510k_1_
- removed R11: 91k 1%, Resistor_SMD:R_0402_1005Metric, symbol nomiq:R11_91k_1_
- removed R12: 100k, Resistor_SMD:R_0402_1005Metric, symbol nomiq:R12_100k
- removed TP2: TP, TestPoint:TestPoint_Pad_D1.0mm, symbol nomiq:TP2_TP
- C1, C3, C4, C6: footprint Capacitor_SMD:C_0603_1608Metric -> nomiq:C_0603_1608Metric
- C10, C2, C5, C9: footprint Capacitor_SMD:C_0402_1005Metric -> nomiq:C_0402_1005Metric
- C11, C7, C8: footprint Capacitor_SMD:C_0805_2012Metric -> nomiq:C_0805_2012Metric
- D1: footprint Package_TO_SOT_SMD:SOT-23-6 -> nomiq:SOT-23-6; PadMap unverified -> datasheet
- D2: footprint Diode_SMD:D_SOD-123F -> nomiq:D_SOD-123F; PadMap unverified -> datasheet
- J1: footprint Connector_USB:USB_C_Receptacle_GCT_USB4105-xx-A_16P_TopMnt_Horizontal -> nomiq:USB_C_Receptacle_GCT_USB4105-xx-A_16P_TopMnt_Horizontal; PadMap unverified -> datasheet
- J2: footprint Connector_JST:JST_PH_S3B-PH-SM4-TB_1x03-1MP_P2.00mm_Horizontal -> nomiq:JST_PH_S3B-PH-SM4-TB_1x03-1MP_P2.00mm_Horizontal; PadMap unverified -> datasheet
- L1: value 0.47uH -> 2.2uH; footprint Inductor_SMD:L_Coilcraft_XFL4015 -> nomiq:L_Taiyo-Yuden_NR-40xx; symbol nomiq:L1_0_47uH -> nomiq:L1_2_2uH; MPN Coilcraft XFL4015-471MEB -> Taiyo Yuden NRS4018T2R2MDGJ; Verify yes -> (none)
- R1, R13, R2, R7, R8, R9: footprint Resistor_SMD:R_0402_1005Metric -> nomiq:R_0402_1005Metric
- R3: footprint Resistor_SMD:R_0402_1005Metric -> nomiq:R_0402_1005Metric; Verify yes -> (none)
- R4: value 1.05k 1% -> 1.13k 1%; footprint Resistor_SMD:R_0402_1005Metric -> nomiq:R_0402_1005Metric; symbol nomiq:R4_1_05k_1_ -> nomiq:R4_1_13k_1_; Verify yes -> (none)
- R5: value 5.36k 1% -> 2.94k 1%; footprint Resistor_SMD:R_0402_1005Metric -> nomiq:R_0402_1005Metric; symbol nomiq:R5_5_36k_1_ -> nomiq:R5_2_94k_1_; Verify yes -> (none)
- R6: value 46.4k 1% -> 37.4k 1%; footprint Resistor_SMD:R_0402_1005Metric -> nomiq:R_0402_1005Metric; symbol nomiq:R6_46_4k_1_ -> nomiq:R6_37_4k_1_; Verify yes -> (none)
- TP1, TP3, TP4, TP5, TP6, TP7: footprint TestPoint:TestPoint_Pad_D1.0mm -> nomiq:TestPoint_Pad_D1.0mm
- U10: value TPS63802 -> TPS63001; footprint Package_SON:Texas_VSON-HR-10_3x2mm_P0.5mm -> nomiq:Texas_S-PVSON-N10; symbol nomiq:U10_TPS63802 -> nomiq:U10_TPS63001; MPN TI TPS63802DLAR -> TI TPS63001DRCR; PadMap unverified -> datasheet; Verify yes -> (none)
- U14: footprint Package_TO_SOT_SMD:SOT-23-6 -> nomiq:SOT-23-6; PadMap unverified -> datasheet; Verify yes -> (none)
- U8: footprint Package_DFN_QFN:VQFN-16-1EP_3x3mm_P0.5mm_EP1.6x1.6mm -> nomiq:VQFN-16-1EP_3x3mm_P0.5mm_EP1.6x1.6mm; PadMap unverified -> datasheet; Verify yes -> (none)
- U9: footprint Package_DFN_QFN:TDFN-8-1EP_2x2mm_P0.5mm_EP0.8x1.2mm -> nomiq:TDFN-8-1EP_2x2mm_P0.5mm_EP0.8x1.2mm; PadMap unverified -> datasheet; Verify yes -> (none)
Connections:
- net BB_FB is gone; now on net VSYS: U10.8 (VINA)
- net PWR_GOOD is gone; now on net GND: U10.9 (GND)
- net BAT_NTC: now also U8.1 (TS); no longer U8.5 (TS)
- net BB_L1: now also U10.4 (L1); no longer U10.5 (L1)
- net BB_L2: now also U10.2 (L2); no longer U10.6 (L2)
- net CHG_ILIM: now also U8.12 (ILIM); no longer U8.7 (ILIM)
- net CHG_ISET: now also U8.16 (ISET); no longer U8.6 (ISET)
- net CHG_ITERM: now also U8.15 (ITERM); no longer U8.8 (ITERM)
- net CHG_STAT_N: now also U8.9 (CHG); no longer U8.13 (CHG)
- net CHG_TMR: now also U8.14 (TMR); no longer U8.9 (TMR)
- net GND: now also D1.2 (GND), D2.2 (A), J1.A1 (GND), J1.A12 (GND), J1.B1 (GND), J1.B12 (GND), J1.SH (SHIELD), J2.MP, U10.11 (EP), U10.7 (PS), U14.2 (GND), U8.17 (EP), U8.6 (EN1), U8.8 (VSS); no longer D1.6 (GND), D2.1 (A), J1.11 (SHIELD), J1.2 (GND), U10.4 (GND), U14.4 (GND), U8.10 (CE), U8.11 (EN1), U8.15 (EP)
- net J1_CC1: now also J1.A5 (CC1); no longer J1.3 (CC1)
- net J1_CC2: now also J1.B5 (CC2); no longer J1.4 (CC2)
- net PGOOD_N: now also U8.7 (PGOOD); no longer U8.14 (PGOOD)
- net STT_CT: now also U14.4 (CT); no longer U14.5 (CT)
- net USB_DN: now also D1.3 (IO2), J1.A7 (DN1), J1.B7 (DN2); no longer D1.2 (IO2), J1.6 (DN1), J1.8 (DN2)
- net USB_DN_MCU: now also D1.4 (IO3); no longer D1.3 (IO3)
- net USB_DP: now also J1.A6 (DP1), J1.B6 (DP2); no longer J1.5 (DP1), J1.7 (DP2)
- net USB_DP_MCU: now also D1.6 (IO4); no longer D1.4 (IO4)
- net V3V3: now also U10.1 (VOUT), U10.10 (FB); no longer U10.7 (VOUT)
- net VBAT: now also U8.2 (BAT)
- net VBUS: now also D2.1 (K), J1.A4 (VBUS), J1.A9 (VBUS), J1.B4 (VBUS), J1.B9 (VBUS), U8.13 (IN); no longer D2.2 (K), J1.1 (VBUS), U8.1 (IN)
- net VSTT: now also U14.5 (QOD); no longer U14.2 (VOUT)
- net VSYS: now also U10.5 (VIN), U10.6 (EN), U8.10 (OUT), U8.11 (OUT), U8.5 (EN2); no longer U10.1 (VIN), U10.2 (EN), U8.12 (EN2), U8.2 (OUT)
Other:
- moved on the sheet: C1, C10, C11, C2, C3, C4, C5, C6, C7, C8, C9, D1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
