File: hardware/kicad/nomiq/02_mcu.kicad_sch (KiCad schematic)
At the start: 18 parts, among them J3 TC2030-IDC-NL, SW1 RESET, SW2 BOOT, U1 ESP32-S3-WROOM-1-N16R8, U4 TCA9535

Commit message: feat(sch): verified pad maps and project footprint library for all 138 parts
- fplib.py: 36 footprints from the KiCad library / Espressif library (+ TFT module),
  written to lib/nomiq.pretty and checked (make tools)
- nomiq_hw.py: per-part datasheet pin->pad maps; gen_kicad checks every pad exists
  and every copper pad is mapped (0 unverified parts)
- TPS63802 -> TPS63001 (fixed 3.3 V, KiCad DRC land pattern); BQ24074 RILIM/ITERM/TMR
  corrected to datasheet constants; TCXO 1.8 V (E) variant to match DIO3 setting
- RF blocks expanded into discrete choke, 2-section low-pass, lattice balun, DC blocks
  (PE4259 ports must be DC-free) and DNP pi tuning pads
- Display: 14-pin ILI9341 module, high-side P-FET backlight switch; microSD detect pins,
  connector mounting pads, MAX98357A NC pads

REQ-PCB-001, REQ-PCB-007

Co-Authored-By: Claude Opus 5.5 <noreply@anthropic.com>
Claude-Session: https://claude.ai/code/session_01HafD3UN2tDPG8DjCdm2PVK
Parts:
- C20, C22, C23: footprint Capacitor_SMD:C_0402_1005Metric -> nomiq:C_0402_1005Metric
- C21: footprint Capacitor_SMD:C_0805_2012Metric -> nomiq:C_0805_2012Metric
- J3: footprint Connector:Tag-Connect_TC2030-IDC-NL_2x03_P1.27mm_Vertical -> nomiq:Tag-Connect_TC2030-IDC-NL_2x03_P1.27mm_Vertical
- R20, R21, R22, R23, R24, R25: footprint Resistor_SMD:R_0402_1005Metric -> nomiq:R_0402_1005Metric
- SW1, SW2: footprint Button_Switch_SMD:Panasonic_EVQPUL_EVQPUC -> nomiq:SW_SPST_PTS810; MPN Panasonic EVQ-P7A01P -> C&K PTS810 SJM 250 SMTR LFS
- TP10, TP8, TP9: footprint TestPoint:TestPoint_Pad_D1.0mm -> nomiq:TestPoint_Pad_D1.0mm
- U1: footprint RF_Module:ESP32-S3-WROOM-1 -> nomiq:ESP32-S3-WROOM-1
- U4: footprint Package_SO:TSSOP-24_4.4x7.8mm_P0.65mm -> nomiq:TSSOP-24_4.4x7.8mm_P0.65mm; PadMap unverified -> datasheet
Connections:
- net AMP_SD_N: now also U4.17 (P14); no longer U4.21 (P14)
- net BTN_BACK_N: now also U4.7 (P03); no longer U4.12 (P03)
- net BTN_CAMERA_N: now also U4.9 (P05); no longer U4.14 (P05)
- net BTN_DOWN_N: now also U4.5 (P01); no longer U4.10 (P01)
- net BTN_RECORD_N: now also U4.8 (P04); no longer U4.13 (P04)
- net BTN_SELECT_N: now also U4.6 (P02); no longer U4.11 (P02)
- net BTN_UP_N: now also U4.4 (P00); no longer U4.9 (P00)
- net CAM_PWDN: now also U4.15 (P12); no longer U4.19 (P12)
- net CAM_PWR_EN: now also U4.19 (P16); no longer U4.23 (P16)
- net CAM_RESET_N: now also U4.16 (P13); no longer U4.20 (P13)
- net CHG_STAT_N: now also U4.10 (P06); no longer U4.15 (P06)
- net FG_ALRT_N: now also U4.20 (P17); no longer U4.24 (P17)
- net GND: now also U4.12 (GND), U4.21 (A0), U4.3 (A2); no longer U4.6 (A0), U4.7 (A1), U4.8 (A2)
- net I2C_SCL: now also U4.22 (SCL); no longer U4.4 (SCL)
- net I2C_SDA: now also U4.23 (SDA); no longer U4.3 (SDA)
- net IOX_INT_N: now also U4.1 (INT); no longer U4.5 (INT)
- net LCD_RST_N: now also U4.14 (P11); no longer U4.18 (P11)
- net LORA_NRST: now also U4.13 (P10); no longer U4.17 (P10)
- net SD_DETECT_N: now also U4.11 (P07); no longer U4.16 (P07)
- net STT_EN: now also U4.18 (P15); no longer U4.22 (P15)
- net V3V3: now also U4.24 (VCC); no longer U4.1 (VCC)
