File: hardware/kicad/nomiq/03_radio.kicad_sch (KiCad schematic)
At the start: 19 parts, among them J4 u.FL, U2 SX1262, U3 PE4259, Y1 TCXO 32 MHz 1.8 V ±2 ppm

Commit message: feat(sch): verified pad maps and project footprint library for all 138 parts
- fplib.py: 36 footprints from the KiCad library / Espressif library (+ TFT module),
  written to lib/nomiq.pretty and checked (make tools)
- nomiq_hw.py: per-part datasheet pin->pad maps; gen_kicad checks every pad exists
  and every copper pad is mapped (0 unverified parts)
- TPS63802 -> TPS63001 (fixed 3.3 V, KiCad DRC land pattern); BQ24074 RILIM/ITERM/TMR
  corrected to datasheet constants; TCXO 1.8 V (E) variant to match DIO3 setting
- RF blocks expanded into discrete choke, 2-section low-pass, lattice balun, DC blocks
  (PE4259 ports must be DC-free) and DNP pi tuning pads
- Display: 14-pin ILI9341 module, high-side P-FET backlight switch; microSD detect pins,
  connector mounting pads, MAX98357A NC pads

REQ-PCB-001, REQ-PCB-007

Co-Authored-By: Claude Opus 5.5 <noreply@anthropic.com>
Claude-Session: https://claude.ai/code/session_01HafD3UN2tDPG8DjCdm2PVK
Parts:
- removed FL1: PA match + harmonic filter (ref design), symbol nomiq:FL1_PA_match___harmonic_filt
- removed FL2: RX balun / match (ref design), symbol nomiq:FL2_RX_balun___match__ref_de
- removed FL3: Antenna π-match (tuning), symbol nomiq:FL3_Antenna___match__tuning_
- added C36: 4.7pF, nomiq:C_0402_1005Metric, symbol nomiq:C36_4_7pF
- added C37: 6.8pF, nomiq:C_0402_1005Metric, symbol nomiq:C37_6_8pF
- added C38: 3.3pF, nomiq:C_0402_1005Metric, symbol nomiq:C38_3_3pF
- added C39: 47pF, nomiq:C_0402_1005Metric, symbol nomiq:C39_47pF
- added C43: 47pF, nomiq:C_0402_1005Metric, symbol nomiq:C43_47pF
- added C44: 2.7pF, nomiq:C_0402_1005Metric, symbol nomiq:C44_2_7pF
- added C45: 2.7pF, nomiq:C_0402_1005Metric, symbol nomiq:C45_2_7pF
- added C46: DNP, nomiq:C_0402_1005Metric, symbol nomiq:C46_DNP
- added C47: 100pF, nomiq:C_0402_1005Metric, symbol nomiq:C47_100pF
- added C48: DNP, nomiq:C_0402_1005Metric, symbol nomiq:C48_DNP
- added L3: 47nH, nomiq:L_0402_1005Metric, symbol nomiq:L3_47nH
- added L4: 12nH, nomiq:L_0402_1005Metric, symbol nomiq:L4_12nH
- added L5: 12nH, nomiq:L_0402_1005Metric, symbol nomiq:L5_12nH
- added L6: 27nH, nomiq:L_0402_1005Metric, symbol nomiq:L6_27nH
- added L7: 27nH, nomiq:L_0402_1005Metric, symbol nomiq:L7_27nH
- C30, C31, C32, C34, C35: footprint Capacitor_SMD:C_0402_1005Metric -> nomiq:C_0402_1005Metric
- C33: footprint Capacitor_SMD:C_0603_1608Metric -> nomiq:C_0603_1608Metric
- D3: footprint Diode_SMD:D_0201_0603Metric -> nomiq:D_0201_0603Metric; PadMap unverified -> datasheet
- J4: footprint Connector_Coaxial:U.FL_Hirose_U.FL-R-SMT-1_Vertical -> nomiq:U.FL_Hirose_U.FL-R-SMT-1_Vertical; PadMap unverified -> datasheet
- L2: footprint Inductor_SMD:L_0805_2012Metric -> nomiq:L_0805_2012Metric
- R30, R31: footprint Resistor_SMD:R_0402_1005Metric -> nomiq:R_0402_1005Metric
- TP11, TP12: footprint TestPoint:TestPoint_Pad_D1.0mm -> nomiq:TestPoint_Pad_D1.0mm
- U2: footprint Package_DFN_QFN:QFN-24-1EP_4x4mm_P0.5mm_EP2.6x2.6mm -> nomiq:QFN-24-1EP_4x4mm_P0.5mm_EP2.6x2.6mm; Verify yes -> (none)
- U3: footprint Package_TO_SOT_SMD:SOT-363_SC-70-6 -> nomiq:SOT-363_SC-70-6; PadMap unverified -> datasheet; Verify yes -> (none)
- Y1: footprint Oscillator:Oscillator_SMD_EuroQuartz_XO32-4Pin_3.2x2.5mm -> nomiq:Crystal_SMD_2016-4Pin_2.0x1.6mm; MPN Epson TG2016SMN 32.0000M-MCGNNM3 -> Epson TG2016SMN 32.0000M-ECGNNM3; PadMap unverified -> datasheet; Verify yes -> (none)
Connections:
- net GND: now also D3.2 (A), U3.2 (GND), C36.2, C37.2, C38.2, C45.2, C46.2, C48.2, L7.2; no longer D3.1 (A), U3.6 (GND)
- net RF_ANT: now also U3.5 (RFC), C46.1, C47.1; no longer U3.3 (RFC)
- net RF_ANT_CONN: now also D3.1 (K), C47.2, C48.1; no longer D3.2 (K)
- net RF_RX: now also U3.3 (RF2), C43.1; no longer U3.2 (RF2)
- net RF_TX: now also C39.2
- net SX_RFI_N: now also C45.1, L6.2
- net SX_RFI_P: now also C44.2, L7.1
- net SX_RFO: now also C36.1, L3.2, L4.1
- net SX_VR_PA: now also L3.1
- net TCXO_VCC: now also Y1.4 (VCC); no longer Y1.1 (VCC)
- net V3V3: now also U3.6 (VDD); no longer U3.5 (VDD)
- new net RX_IN: C43.2, C44.1, L6.1
- new net TX_N1: C37.1, L4.2, L5.1
- new net TX_N2: C38.1, C39.1, L5.2
Other:
- moved on the sheet: D3, L2, R30, R31, TP11, TP12
