File: hardware/kicad/nomiq/05_camera.kicad_sch (KiCad schematic)
At the start: 10 parts, among them J6 OV2640 24P FPC 0.5 mm, U12 TLV75528 (2.8 V), U13 TLV75512 (1.2 V), U15 TPS22918 (cam 3V3)

Commit message: feat(sch): verified pad maps and project footprint library for all 138 parts
- fplib.py: 36 footprints from the KiCad library / Espressif library (+ TFT module),
  written to lib/nomiq.pretty and checked (make tools)
- nomiq_hw.py: per-part datasheet pin->pad maps; gen_kicad checks every pad exists
  and every copper pad is mapped (0 unverified parts)
- TPS63802 -> TPS63001 (fixed 3.3 V, KiCad DRC land pattern); BQ24074 RILIM/ITERM/TMR
  corrected to datasheet constants; TCXO 1.8 V (E) variant to match DIO3 setting
- RF blocks expanded into discrete choke, 2-section low-pass, lattice balun, DC blocks
  (PE4259 ports must be DC-free) and DNP pi tuning pads
- Display: 14-pin ILI9341 module, high-side P-FET backlight switch; microSD detect pins,
  connector mounting pads, MAX98357A NC pads

REQ-PCB-001, REQ-PCB-007

Co-Authored-By: Claude Opus 5.5 <noreply@anthropic.com>
Claude-Session: https://claude.ai/code/session_01HafD3UN2tDPG8DjCdm2PVK
Parts:
- C50, C51, C52, C53: footprint Capacitor_SMD:C_0402_1005Metric -> nomiq:C_0402_1005Metric
- J6: footprint Connector_FFC-FPC:Hirose_FH12-24S-0.5SH_1x24-1MP_P0.50mm_Horizontal -> nomiq:Hirose_FH12-24S-0.5SH_1x24-1MP_P0.50mm_Horizontal; PadMap unverified -> datasheet
- R50, R51: footprint Resistor_SMD:R_0402_1005Metric -> nomiq:R_0402_1005Metric
- U12, U13: footprint Package_TO_SOT_SMD:SOT-23-5 -> nomiq:SOT-23-5; PadMap unverified -> datasheet
- U15: footprint Package_TO_SOT_SMD:SOT-23-6 -> nomiq:SOT-23-6; PadMap unverified -> datasheet
Connections:
- net CAM_CT: now also U15.4 (CT); no longer U15.5 (CT)
- net CAM_D0: now also J6.19 (Y2); no longer J6.18 (Y2)
- net CAM_D1: now also J6.21 (Y3); no longer J6.20 (Y3)
- net CAM_D2: now also J6.22 (Y4); no longer J6.21 (Y4)
- net CAM_D3: now also J6.20 (Y5); no longer J6.19 (Y5)
- net CAM_D4: now also J6.18 (Y6); no longer J6.17 (Y6)
- net CAM_D5: now also J6.16 (Y7); no longer J6.15 (Y7)
- net CAM_D6: now also J6.14 (Y8); no longer J6.13 (Y8)
- net CAM_D7: now also J6.12 (Y9); no longer J6.11 (Y9)
- net CAM_HREF: now also J6.9 (HREF); no longer J6.8 (HREF)
- net CAM_PCLK: now also J6.17 (PCLK); no longer J6.16 (PCLK)
- net CAM_PWDN: now also J6.8 (PWDN); no longer J6.7 (PWDN)
- net CAM_RESET_N: now also J6.6 (RESETB); no longer J6.5 (RESETB)
- net CAM_VSYNC: now also J6.7 (VSYNC); no longer J6.6 (VSYNC)
- net CAM_XCLK: now also J6.13 (XCLK); no longer J6.12 (XCLK)
- net GND: now also J6.15 (DGND), J6.2 (AGND), J6.MP, U12.2 (GND), U13.2 (GND), U15.2 (GND); no longer J6.1 (AGND), J6.14 (DGND), U12.3 (GND), U13.3 (GND), U15.4 (GND)
- net I2C_SCL: now also J6.5 (SCL); no longer J6.4 (SCL)
- net I2C_SDA: now also J6.3 (SDA); no longer J6.2 (SDA)
- net VCAM_1V2: now also J6.10 (DVDD), U13.5 (OUT); no longer J6.9 (DVDD), U13.4 (OUT)
- net VCAM_2V8: now also J6.4 (AVDD), U12.5 (OUT); no longer J6.3 (AVDD), U12.4 (OUT)
- net VCAM_3V3: now also J6.11 (DOVDD), U12.3 (EN), U13.3 (EN), U15.5 (QOD); no longer J6.10 (DOVDD), U12.2 (EN), U13.2 (EN), U15.2 (VOUT)
Other:
- moved on the sheet: C50, C51, C52, C53, R50, R51, U15
