File: hardware/kicad/nomiq/07_ui.kicad_sch (KiCad schematic)
At the start: 19 parts, among them SW3 button (front), SW4 button (front), SW5 button (front), SW6 button (front), SW7 button (left side), SW8 button (right side), SW9 POWER (ship-mode / wake)

Commit message: feat(sch): verified pad maps and project footprint library for all 138 parts
- fplib.py: 36 footprints from the KiCad library / Espressif library (+ TFT module),
  written to lib/nomiq.pretty and checked (make tools)
- nomiq_hw.py: per-part datasheet pin->pad maps; gen_kicad checks every pad exists
  and every copper pad is mapped (0 unverified parts)
- TPS63802 -> TPS63001 (fixed 3.3 V, KiCad DRC land pattern); BQ24074 RILIM/ITERM/TMR
  corrected to datasheet constants; TCXO 1.8 V (E) variant to match DIO3 setting
- RF blocks expanded into discrete choke, 2-section low-pass, lattice balun, DC blocks
  (PE4259 ports must be DC-free) and DNP pi tuning pads
- Display: 14-pin ILI9341 module, high-side P-FET backlight switch; microSD detect pins,
  connector mounting pads, MAX98357A NC pads

REQ-PCB-001, REQ-PCB-007

Co-Authored-By: Claude Opus 5.5 <noreply@anthropic.com>
Claude-Session: https://claude.ai/code/session_01HafD3UN2tDPG8DjCdm2PVK
Parts:
- D70, D71, D72, D73, D74, D75: footprint Diode_SMD:D_SOD-882 -> nomiq:D_SOD-882; PadMap unverified -> datasheet
- R70, R71, R72, R73, R74, R75: footprint Resistor_SMD:R_0402_1005Metric -> nomiq:R_0402_1005Metric
- SW3, SW4, SW5, SW6: footprint (none) -> nomiq:SW_SPST_PTS810; MPN C&K PTS526 -> C&K PTS810 SJM 250 SMTR LFS
- SW7, SW8, SW9: footprint (none) -> nomiq:SW_SPST_EVQP7A
Connections:
- net BTN_BACK_N: now also D73.1 (K); no longer D73.2 (K)
- net BTN_CAMERA_N: now also D75.1 (K); no longer D75.2 (K)
- net BTN_DOWN_N: now also D71.1 (K); no longer D71.2 (K)
- net BTN_RECORD_N: now also D74.1 (K); no longer D74.2 (K)
- net BTN_SELECT_N: now also D72.1 (K); no longer D72.2 (K)
- net BTN_UP_N: now also D70.1 (K); no longer D70.2 (K)
- net GND: now also D70.2 (A), D71.2 (A), D72.2 (A), D73.2 (A), D74.2 (A), D75.2 (A); no longer D70.1 (A), D71.1 (A), D72.1 (A), D73.1 (A), D74.1 (A), D75.1 (A)
