File: hardware/kicad/nomiq/08_stt.kicad_sch (KiCad schematic)
At the start: 1 part, among them J9 STT SoM interface 2x5 1.27 mm

Commit message: feat(sch): verified pad maps and project footprint library for all 138 parts
- fplib.py: 36 footprints from the KiCad library / Espressif library (+ TFT module),
  written to lib/nomiq.pretty and checked (make tools)
- nomiq_hw.py: per-part datasheet pin->pad maps; gen_kicad checks every pad exists
  and every copper pad is mapped (0 unverified parts)
- TPS63802 -> TPS63001 (fixed 3.3 V, KiCad DRC land pattern); BQ24074 RILIM/ITERM/TMR
  corrected to datasheet constants; TCXO 1.8 V (E) variant to match DIO3 setting
- RF blocks expanded into discrete choke, 2-section low-pass, lattice balun, DC blocks
  (PE4259 ports must be DC-free) and DNP pi tuning pads
- Display: 14-pin ILI9341 module, high-side P-FET backlight switch; microSD detect pins,
  connector mounting pads, MAX98357A NC pads

REQ-PCB-001, REQ-PCB-007

Co-Authored-By: Claude Opus 5.5 <noreply@anthropic.com>
Claude-Session: https://claude.ai/code/session_01HafD3UN2tDPG8DjCdm2PVK
Parts:
- J9: footprint (none) -> nomiq:PinHeader_2x05_P1.27mm_Vertical_SMD; PadMap unverified -> datasheet
Changed lines of the file:
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@@
 (kicad_sch (version 20231120) (generator "nomiq_gen") (generator_version "8.0") (paper "A2")
 (title_block (title "Nomiq A0 — 08_stt") (rev "A0") (comment 1 "Generated from hardware/design/nomiq_hw.py - edit the spec, then regenerate"))
-(symbol (lib_id "nomiq:J9_STT_SoM_interface_2x5_1_") (at 86.36 55.88 0) (unit 1) (exclude_from_sim no) (in_bom yes) (on_board yes) (dnp no) (property "Reference" "J9" (at 86.36 45.72 0) (effects (font (size 1.27 1.27)))) (property "Value" "STT SoM interface 2x5 1.27 mm" (at 86.36 66.04 0) (effects (font (size 1.27 1.27)))) (property "Footprint" "" (at 86.36 55.88 0) (effects (font (size 1.27 1.27)) (hide yes))) (property "Datasheet" "" (at 86.36 55.88 0) (effects (font (size 1.27 1.27)) (hide yes))) (property "MPN" "Samtec FTSH-105-01-L-DV" (at 86.36 55.88 0) (effects (font (size 1.27 1.27)) (hide yes))) (property "Verify" "" (at 86.36 55.88 0) (effects (font (size 1.27 1.27)) (hide yes))) (property "PadMap" "unverified" (at 86.36 55.88 0) (effects (font (size 1.27 1.27)) (hide yes))) (pin "1") (pin "2") (pin "3") (pin "4") (pin "5") (pin "6") (pin "7") (pin "8") (pin "9") (pin "10") (instances (project "nomiq" (path "/22a78807-b768-5690-bf1c-caee3a2f8ff0/0e925b6e-e453-5b40-b9a2-cb0fdf22bfc4" (reference "J9") (unit 1)))))
+(symbol (lib_id "nomiq:J9_STT_SoM_interface_2x5_1_") (at 86.36 55.88 0) (unit 1) (exclude_from_sim no) (in_bom yes) (on_board yes) (dnp no) (property "Reference" "J9" (at 86.36 45.72 0) (effects (font (size 1.27 1.27)))) (property "Value" "STT SoM interface 2x5 1.27 mm" (at 86.36 66.04 0) (effects (font (size 1.27 1.27)))) (property "Footprint" "nomiq:PinHeader_2x05_P1.27mm_Vertical_SMD" (at 86.36 55.88 0) (effects (font (size 1.27 1.27)) (hide yes))) (property "Datasheet" "" (at 86.36 55.88 0) (effects (font (size 1.27 1.27)) (hide yes))) (property "MPN" "Samtec FTSH-105-01-L-DV" (at 86.36 55.88 0) (effects (font (size 1.27 1.27)) (hide yes))) (property "Verify" "" (at 86.36 55.88 0) (effects (font (size 1.27 1.27)) (hide yes))) (property "PadMap" "datasheet" (at 86.36 55.88 0) (effects (font (size 1.27 1.27)) (hide yes))) (pin "1") (pin "2") (pin "3") (pin "4") (pin "5") (pin "6") (pin "7") (pin "8") (pin "9") (pin "10") (instances (project "nomiq" (path "/22a78807-b768-5690-bf1c-caee3a2f8ff0/0e925b6e-e453-5b40-b9a2-cb0fdf22bfc4" (reference "J9") (unit 1)))))
 (wire (pts (xy 68.58 50.80) (xy 66.04 50.80)) (stroke (width 0) (type default)))
 (global_label "VSTT" (shape bidirectional) (at 66.04 50.80 180) (fields_autoplaced yes) (effects (font (size 1.27 1.27)) (justify right)) (property "Intersheetrefs" "${INTERSHEET_REFS}" (at 66.04 50.80 0) (effects (font (size 1.27 1.27)) (hide yes))))
